Commit message: change xacro file so robot can spawn at gazebo and create custom teleop for control jupiter robot

File: src/jupiterobot2_arm_description/urdf/jupiterobot2_arm_gazebo.xacro (robot description, xacro)
@@ -1,47 +1,56 @@
 <?xml version="1.0"?>
 <robot xmlns:xacro="http://ros.org/wiki/xacro">
-  <!-- Transmission macro -->
-  <xacro:macro name="SimpleTransmissionPosition" params="joint n">
-    <transmission name="tran${n}">
-      <type>transmission_interface/SimpleTransmission</type>
-      <joint name="${joint}">
-        <hardwareInterface>hardware_interface/PositionJointInterface</hardwareInterface>
-      </joint>
-      <actuator name="motor${n}">
-        <hardwareInterface>hardware_interface/PositionJointInterface</hardwareInterface>
-        <mechanicalReduction>1</mechanicalReduction>
-      </actuator>
-    </transmission>
-  </xacro:macro>
-  <!-- Transmission macro -->
-  <xacro:macro name="SimpleTransmissionEffort" params="joint n">
-    <transmission name="tran${n}">
-      <type>transmission_interface/SimpleTransmission</type>
-      <joint name="${joint}">
-        <hardwareInterface>hardware_interface/EffortJointInterface</hardwareInterface>
-      </joint>
-      <actuator name="motor${n}">
-        <hardwareInterface>hardware_interface/EffortJointInterface</hardwareInterface>
-        <mechanicalReduction>1</mechanicalReduction>
-      </actuator>
-    </transmission>
-  </xacro:macro>
-  <!-- Transmission 1 -->
-  <xacro:SimpleTransmissionPosition n="1" joint="arm1_joint" />
-  <!-- Transmission 2 -->
-  <xacro:SimpleTransmissionPosition n="2" joint="arm2_joint" />
-  <!-- Transmission 3 -->
-  <xacro:SimpleTransmissionPosition n="3" joint="arm3_joint" />
-  <!-- Transmission 4 -->
-  <xacro:SimpleTransmissionPosition n="4" joint="arm4_joint" />
-  <!-- Transmission 5 -->
-  <xacro:SimpleTransmissionPosition n="5" joint="gripper_joint" />
-  <!-- ros_control plugin -->
+  <ros2_control name="GazeboSystem" type="system">
+    <hardware>
+      <plugin>gazebo_ros2_control/GazeboSystem</plugin>
+    </hardware>
+    <joint name="arm1_joint">
+      <command_interface name="position" />
+      <state_interface name="position" />
+      <state_interface name="velocity" />
+      <state_interface name="effort" />
+    </joint>
+    <joint name="arm2_joint">
+      <command_interface name="position" />
+      <state_interface name="position" />
+      <state_interface name="velocity" />
+      <state_interface name="effort" />
+    </joint>
+    <joint name="arm3_joint">
+      <command_interface name="position" />
+      <state_interface name="position" />
+      <state_interface name="velocity" />
+      <state_interface name="effort" />
+    </joint>
+    <joint name="arm4_joint">
+      <command_interface name="position" />
+      <state_interface name="position" />
+      <state_interface name="velocity" />
+      <state_interface name="effort" />
+    </joint>
+    <joint name="gripper_joint">
+      <command_interface name="position" />
+      <state_interface name="position" />
+      <state_interface name="velocity" />
+      <state_interface name="effort" />
+    </joint>
+  <joint name="gripper_joint">
+      <command_interface name="position" />
+      <state_interface name="position" />
+      <state_interface name="velocity" />
+      <state_interface name="effort" />
+    </joint>
+  <joint name="head_joint">
+    <command_interface name="position" />
+    <state_interface name="position" />
+    <state_interface name="velocity" />
+    <state_interface name="effort" />
+  </joint>
+  </ros2_control>
   <gazebo>
-    <plugin name="gazebo_ros_control" filename="libgazebo_ros_control.so">
-      <controlPeriod>0.001</controlPeriod>
-      <robotNamespace>/</robotNamespace>
-      <robotSimType>gazebo_ros_control/DefaultRobotHWSim</robotSimType>
-      <legacyModeNS>true</legacyModeNS>
+    <plugin name="gazebo_ros2_control" filename="libgazebo_ros2_control.so">
+      <robot_param>robot_description</robot_param>
+      <robot_param_node>robot_state_publisher</robot_param_node>
+      <parameters>$(find jupiterobot2_gazebo)/config/controllers.yaml</parameters>
     </plugin>
   </gazebo>

File: src/jupiterobot2_description/urdf/jupiter2_gazebo.xacro (robot description, xacro)
@@ -8,146 +8,67 @@
   </gazebo>
   <gazebo reference="wheel_left_link">
-    <mu1>1</mu1>
-    <mu2>1</mu2>
+    <mu1>1.0</mu1>
+    <mu2>1.0</mu2>
     <kp>1e6</kp>
     <kd>1e3</kd>
     <minDepth>0.001</minDepth>
-    <maxVel>1</maxVel>
+    <maxVel>1.0</maxVel>
     <material>Gazebo/FlatBlack</material>
   </gazebo>
   <gazebo reference="wheel_right_link">
-    <mu1>1</mu1>
-    <mu2>1</mu2>
+    <mu1>1.0</mu1>
+    <mu2>1.0</mu2>
     <kp>1e6</kp>
     <kd>1e3</kd>
     <minDepth>0.001</minDepth>
-    <maxVel>1</maxVel>
+    <maxVel>1.0</maxVel>
     <material>Gazebo/FlatBlack</material>
   </gazebo>
   <gazebo reference="caster_back_right_link">
-    <mu1>0.01</mu1>
-    <mu2>0.01</mu2>
+    <mu1>0.0</mu1>
+    <mu2>0.0</mu2>
     <kp>1e6</kp>
     <kd>1e3</kd>
-    <minDepth>0.001</minDepth>
-    <maxVel>1</maxVel>
     <material>Gazebo/Grey</material>
   </gazebo>
   <gazebo reference="caster_back_left_link">
-    <mu1>0.01</mu1>
-    <mu2>0.01</mu2>
+    <mu1>0.0</mu1>
+    <mu2>0.0</mu2>
     <kp>1e6</kp>
     <kd>1e3</kd>
-    <minDepth>0.001</minDepth>
-    <maxVel>1</maxVel>
     <material>Gazebo/Grey</material>
+  </gazebo>
+  <gazebo>
+    <plugin name="jupiter2_diff_drive" filename="libgazebo_ros_diff_drive.so">
+      <ros>
+        <remapping>cmd_vel:=cmd_vel</remapping>
+        <remapping>odom:=odom</remapping>
+      </ros>
+      <left_joint>wheel_left_joint</left_joint>
+      <right_joint>wheel_right_joint</right_joint>
+      <wheel_separation>0.287</wheel_separation>
+      <wheel_diameter>0.066</wheel_diameter>
+      <max_wheel_torque>20</max_wheel_torque>
+      <max_wheel_acceleration>1.0</max_wheel_acceleration>
+      <publish_odom>true</publish_odom>
+      <publish_odom_tf>true</publish_odom_tf>
+      <publish_wheel_tf>true</publish_wheel_tf>
+      <odometry_frame>odom</odometry_frame>
+      <robot_base_frame>base_footprint</robot_base_frame>
+    </plugin>
   </gazebo>
   <gazebo reference="imu_link">
     <sensor type="imu" name="imu">
       <always_on>true</always_on>
+      <update_rate>100</update_rate>
       <visualize>$(arg imu_visual)</visualize>
+      <plugin name="imu_plugin" filename="libgazebo_ros_imu_sensor.so">
+        <ros>
+          <remapping>~/out:=imu</remapping>
+        </ros>
+      </plugin>
     </sensor>
     <material>Gazebo/Grey</material>
   </gazebo>
-  <gazebo reference="plate_1_link">
-    <material>Gazebo/Black</material>
-  </gazebo>
-  <gazebo reference="plate_2_link">
-    <material>Gazebo/Black</material>
-  </gazebo>
-  <gazebo reference="plate_3_link">
-    <material>Gazebo/Black</material>
-  </gazebo>
-  <gazebo reference="arrow_link">
-    <material>Gazebo/White</material>
-  </gazebo>
-  <gazebo reference="mic_link">
-    <material>Gazebo/DarkGrey</material>
-  </gazebo>
-  <gazebo reference="estop_link">
-    <material>Gazebo/DarkGrey</material>
-  </gazebo>
-  <gazebo reference="monitor_frame_1_link">
-    <material>Gazebo/DarkGrey</material>
-  </gazebo>
-  <gazebo reference="monitor_frame_2_link">
-    <material>Gazebo/DarkGrey</material>
-  </gazebo>
-  <gazebo reference="monitor_link">
-    <material>Gazebo/FlatBlack</material>
-  </gazebo>
-  <gazebo reference="screen_link">
-    <material>Gazebo/WhiteGlow</material>
-  </gazebo>
-  <gazebo reference="arm_mount_link">
-    <material>Gazebo/DarkGrey</material>
-  </gazebo>
-  <gazebo reference="head_mount_link">
-    <material>Gazebo/DarkGrey</material>
-  </gazebo>
-  <gazebo reference="pipe_200_link">
-    <material>Gazebo/BlackTransparent</material>
-  </gazebo>
-  <gazebo reference="pipe_300_link">
-    <material>Gazebo/BlackTransparent</material>
-  </gazebo>
-  <gazebo reference="cables_link">
-    <material>Gazebo/BlackTransparent</material>
-  </gazebo>
-<!-- change at 9.58 by comented -->
-  <!-- <gazebo>
-    <plugin name="jupiter2_controller" filename="libgazebo_ros_diff_drive.so">
-      <commandTopic>cmd_vel</commandTopic>
-      <odometryTopic>odom</odometryTopic>
-      <odometryFrame>odom</odometryFrame>
-      <odometrySource>world</odometrySource>
-      <publishOdomTF>true</publishOdomTF>
-      <robotBaseFrame>base_footprint</robotBaseFrame>
-      <publishWheelTF>false</publishWheelTF>
-      <publishTf>true</publishTf>
-      <publishWheelJointState>true</publishWheelJointState>
-      <legacyMode>false</legacyMode>
-      <updateRate>30</updateRate>
-      <leftJoint>wheel_left_joint</leftJoint>
-      <rightJoint>wheel_right_joint</rightJoint>
-      <wheelSeparation>0.287</wheelSeparation>
-      <wheelDiameter>0.066</wheelDiameter>
-      <wheelAcceleration>1</wheelAcceleration>
-      <wheelTorque>10</wheelTorque>
-      <rosDebugLevel>na</rosDebugLevel>
-    </plugin>
-  </gazebo> -->
-<!--eweadasdad  -->
-<!-- change at 9.58 by comented -->
-  <!-- <gazebo>
-    <plugin name="imu_plugin" filename="libgazebo_ros_imu.so">
-      <alwaysOn>true</alwaysOn>
-      <bodyName>imu_link</bodyName>
-      <frameName>imu_link</frameName>
-      <topicName>imu</topicName>
-      <serviceName>imu_service</serviceName>
-      <gaussianNoise>0.0</gaussianNoise>
-      <updateRate>0</updateRate>
-      <imu>
-        <noise>
-          <type>gaussian</type>
-          <rate>
-            <mean>0.0</mean>
-            <stddev>2e-4</stddev>
-            <bias_mean>0.0000075</bias_mean>
-            <bias_stddev>0.0000008</bias_stddev>
-          </rate>
-          <accel>
-            <mean>0.0</mean>
-            <stddev>1.7e-2</stddev>
-            <bias_mean>0.1</bias_mean>
-            <bias_stddev>0.001</bias_stddev>
-          </accel>
-        </noise>
-      </imu>
-    </plugin>
-  </gazebo> -->
-<!-- safa -->
-  <!-- $(arg laser_visual) -->
   <gazebo reference="base_scan">
     <material>Gazebo/FlatBlack</material>
@@ -161,11 +82,11 @@
             <samples>360</samples>
             <resolution>1</resolution>
-            <min_angle>-3.14159265359</min_angle>
-            <max_angle>3.14159265359</max_angle>
+            <min_angle>-3.14159</min_angle>
+            <max_angle>3.14159</max_angle>
           </horizontal>
         </scan>
         <range>
           <min>0.234</min>
-          <max>10.0</max>
+          <max>12.0</max>
           <resolution>0.01</resolution>
         </range>
@@ -176,57 +97,17 @@
         </noise>
       </ray>
-      <!-- changed 10.03 pm -->
-      <!-- <plugin name="gazebo_ros_rplidar_a1_controller" filename="libgazebo_ros_laser.so">
-        <topicName>scan</topicName>
-        <frameName>base_scan</frameName>
-      </plugin> -->
-      <!-- DADAS -->
+      <plugin name="gazebo_ros_laser_controller" filename="libgazebo_ros_ray_sensor.so">
+        <ros>
+          <remapping>~/out:=scan</remapping>
+        </ros>
+        <output_type>sensor_msgs/LaserScan</output_type>
+        <frame_name>base_scan</frame_name>
+      </plugin>
     </sensor>
   </gazebo>
-  <gazebo reference="camera_link">
-    <sensor type="depth" name="camera">
-      <always_on>true</always_on>
-      <visualize>$(arg camera_visual)</visualize>
-      <update_rate>20.0</update_rate>
-      <camera>
-          <horizontal_fov>1.0472</horizontal_fov>
-          <image>
-              <width>640</width>
-              <height>480</height>
-              <format>R8G8B8</format>
-          </image>
-          <depth_camera></depth_camera>
-          <clip>
-              <near>0.05</near>
-              <far>8.0</far>
-          </clip>
-      </camera>
-      <!-- 12/1/2026 comennted by 10.04 -->
-      <!-- <plugin name="camera_controller" filename="libgazebo_ros_openni_kinect.so">
-        <baseline>0.1</baseline>
-        <alwaysOn>true</alwaysOn>
-        <updateRate>20.0</updateRate>
-        <cameraName>camera</cameraName>
-        <frameName>camera_depth_optical_frame</frameName>
-        <imageTopicName>color/image_raw</imageTopicName>
-        <depthImageTopicName>depth/image_raw</depthImageTopicName>
-        <pointCloudTopicName>depth/points</pointCloudTopicName>
-        <cameraInfoTopicName>color/camera_info</cameraInfoTopicName>
-        <depthImageCameraInfoTopicName>depth/camera_info</depthImageCameraInfoTopicName>
-        <pointCloudCutoff>0.4</pointCloudCutoff>
-            <hackBaseline>0.07</hackBaseline>
-            <distortionK1>0.0</distortionK1>
-            <distortionK2>0.0</distortionK2>
-            <distortionK3>0.0</distortionK3>
-            <distortionT1>0.0</distortionT1>
-            <distortionT2>0.0</distortionT2>
-        <CxPrime>0.0</CxPrime>
-        <Cx>0.0</Cx>
-        <Cy>0.0</Cy>
-        <focalLength>0</focalLength>
-        <hackBaseline>0</hackBaseline>
-      </plugin> -->
-      <!--  -->
-    </sensor>
-  </gazebo>
+  <gazebo reference="plate_1_link"><material>Gazebo/Black</material></gazebo>
+  <gazebo reference="plate_2_link"><material>Gazebo/Black</material></gazebo>
+  <gazebo reference="plate_3_link"><material>Gazebo/Black</material></gazebo>
+  <gazebo reference="monitor_link"><material>Gazebo/FlatBlack</material></gazebo>
+  <gazebo reference="screen_link"><material>Gazebo/WhiteGlow</material></gazebo>
 </robot>

File: src/jupiterobot2_head_description/urdf/jupiterobot2_head_gazebo.xacro (robot description, xacro)
@@ -1,40 +1,14 @@
 <?xml version="1.0"?>
 <robot xmlns:xacro="http://ros.org/wiki/xacro">
-  <!-- Transmission macro -->
-  <xacro:macro name="SimpleTransmissionPosition" params="joint n">
-    <transmission name="tran${n}">
-      <type>transmission_interface/SimpleTransmission</type>
-      <joint name="${joint}">
-        <hardwareInterface>hardware_interface/PositionJointInterface</hardwareInterface>
-      </joint>
-      <actuator name="motor${n}">
-        <hardwareInterface>hardware_interface/PositionJointInterface</hardwareInterface>
-        <mechanicalReduction>1</mechanicalReduction>
-      </actuator>
-    </transmission>
-  </xacro:macro>
-  <!-- Transmission macro -->
-  <xacro:macro name="SimpleTransmissionEffort" params="joint n">
-    <transmission name="tran${n}">
-      <type>transmission_interface/SimpleTransmission</type>
-      <joint name="${joint}">
-        <hardwareInterface>hardware_interface/EffortJointInterface</hardwareInterface>
-      </joint>
-      <actuator name="motor${n}">
-        <hardwareInterface>hardware_interface/EffortJointInterface</hardwareInterface>
-        <mechanicalReduction>1</mechanicalReduction>
-      </actuator>
-    </transmission>
-  </xacro:macro>
-  <!-- Transmission 6 -->
-  <xacro:SimpleTransmissionPosition n="6" joint="head_joint" />
-  <!-- ros_control plugin -->
-  <!-- <gazebo>
-    <plugin name="gazebo_ros_control" filename="libgazebo_ros_control.so">
-      <controlPeriod>0.001</controlPeriod>
-      <robotNamespace>/</robotNamespace>
-      <robotSimType>gazebo_ros_control/DefaultRobotHWSim</robotSimType>
-      <legacyModeNS>true</legacyModeNS>
-    </plugin>
-  </gazebo> -->
-</robot>
+  <ros2_control name="GazeboHeadSystem" type="system">
+    <hardware>
+      <plugin>gazebo_ros2_control/GazeboSystem</plugin>
+    </hardware>
+    <joint name="head_joint">
+      <command_interface name="position" />
+      <state_interface name="position" />
+      <state_interface name="velocity" />
+      <state_interface name="effort" />
+    </joint>
+  </ros2_control>
+  </robot>
